Commit message: Added rviz functionalities

File: humanoid_robot/urdf/humanoid_robot.urdf.xacro (robot description, xacro)
@@ -4,4 +4,6 @@
      For more information, please see http://wiki.ros.org/sw_urdf_exporter -->
 <robot name="humanoid_robot" xmlns:xacro="http://ros.org/wiki/xacro">
+  <!-- # Add this before base link -->
+<link name="dummy_link"></link>
   <link
     name="base_link">
@@ -44,4 +46,10 @@
     </collision>
   </link>
+  <!-- # Add this after base link -->
+<joint name="dummy_joint" type="fixed">
+    <origin rpy="0 0 0" xyz="0 0 0" />
+    <parent link="dummy_link"/>
+    <child link="base_link"/>
+</joint>
   <link
     name="Hip_Left">
